Commit message: maj -> controle manette

File: src/car_square/model/model.xacro (robot description, xacro)
@@ -50,16 +50,20 @@
                 <joint name="lf_joint">
                         <command_interface name="velocity"/>
+                        <state_interface name="position"/>
                         <state_interface name="velocity"/>
                 </joint>
                 <joint name="rf_joint">
                         <command_interface name="velocity"/>
+                        <state_interface name="position"/>
                         <state_interface name="velocity"/>
                 </joint>
                 <joint name="lb_joint">
                         <command_interface name="velocity"/>
+                        <state_interface name="position"/>
                         <state_interface name="velocity"/>
                 </joint>
                 <joint name="rb_joint">
                         <command_interface name="velocity"/>
+                        <state_interface name="position"/>
                         <state_interface name="velocity"/>
                 </joint>

File: src/car_square/model/model_simu.xacro (robot description, xacro)
@@ -13,5 +13,5 @@
                 <collision>
                         <geometry>
-                        <box size="0.3 0.25 0.05"/>
+                        <box size="${chassis_length} ${chassis_width} ${chassis_height}"/>
                         </geometry>
                         <origin xyz="0 0 ${chassis_offset}" rpy="0 0 0"/>
@@ -19,4 +19,18 @@
                 <xacro:chassis_inertia />
         </link>
+        <link name="visual_front">
+                <visual>
+                        <geometry>
+                        <box size="${chassis_length/8} ${chassis_width/2} ${chassis_height/4}"/>
+                        </geometry>
+                        <origin xyz="${3*chassis_length/8} 0 ${1.5*chassis_offset - chassis_height/8}" rpy="0 0 0"/>
+                        <material name="green"/>
+                </visual>
+        </link>
+        <joint name="visual_front_joint" type="fixed">
+                <parent link="base_link"/>
+                <child link="visual_front"/>
+                <origin xyz="0 0 0" rpy="0 0 0"/>
+        </joint>
         <!-- LINKS ET JOINTS DES ROUES -->
         <xacro:omni_wheel
@@ -53,5 +67,4 @@
                         <state_interface name="position"/>
                         <state_interface name="velocity"/>
-                        <state_interface name="effort"/>
                 </joint>
                 <joint name="rf_joint">
@@ -59,5 +72,4 @@
                         <state_interface name="position"/>
                         <state_interface name="velocity"/>
-                        <state_interface name="effort"/>
                 </joint>
                 <joint name="lb_joint">
@@ -65,5 +77,4 @@
                         <state_interface name="position"/>
                         <state_interface name="velocity"/>
-                        <state_interface name="effort"/>
                 </joint>
                 <joint name="rb_joint">
@@ -71,5 +82,4 @@
                         <state_interface name="position"/>
                         <state_interface name="velocity"/>
-                        <state_interface name="effort"/>
                 </joint>
         </ros2_control>
